Commit message: Task_1: ongoing

File: src/task1/urdf/hola_bot.urdf (robot description, URDF)
Before this commit: robot hola_bot, 2 links, 1 joints
Links:
- added link back_left_wheel, mass 0.062; collision cylinder length=0.02 radius=.03; visual mesh filename=package://hola/meshes/wheel.STL
- added link back_right_wheel, mass 0.062; collision cylinder length=0.02 radius=.03; visual mesh filename=package://hola/meshes/wheel.STL
- link base_link: geometry collision cylinder length=0.005 radius=0.15; visual mesh filename=package://hola/meshes/base_link.STL
- link front_wheel: geometry collision cylinder length=0.02 radius=.03; visual mesh filename=package://hola/meshes/wheel.STL
Joints:
- added joint back_left_joint: type continuous, parent base_link, child back_left_wheel, origin xyz=-0.15154 -0.087275 -0.0335 rpy=0 0 2.05304, axis 0 -1 0, limit effort=5 velocity=5
- added joint back_right_joint: type continuous, parent base_link, child back_right_wheel, origin xyz=0.14044 -0.07927500000000001 -0.0335 rpy=0 0 1.01229, axis 0 -1 0, limit effort=5 velocity=5
