Commit message: made seperate package for hola_bot gazebo

File: src/hola_bot/urdf/hola_bot.urdf (robot description, URDF)
Before this commit: robot hola_bot, 4 links, 3 joints
Links:
- link back_left_wheel: geometry collision cylinder length=0.02 radius=.03; visual mesh filename=package://hola_bot/meshes/wheel.STL
- link back_right_wheel: geometry collision cylinder length=0.02 radius=.03; visual mesh filename=package://hola_bot/meshes/wheel.STL
- link base_link: geometry collision cylinder length=0.005 radius=0.15; visual mesh filename=package://hola_bot/meshes/base_link.STL
- link front_wheel: geometry collision cylinder length=0.02 radius=.03; visual mesh filename=package://hola_bot/meshes/wheel.STL

Commit message: updated hola_bot package

File: src/hola_bot/urdf/hola_bot.urdf (robot description, URDF)
Before this commit: robot hola_bot, 4 links, 3 joints
Links:
- removed link back_left_wheel
- removed link back_right_wheel
- added link left_wheel, mass 0.060; collision cylinder length=0.02 radius=.03; visual mesh filename=package://hola_bot/meshes/wheel.STL
- added link right_wheel, mass 0.060; collision cylinder length=0.02 radius=.03; visual mesh filename=package://hola_bot/meshes/wheel.STL
- link base_link: mass 0.49 -> 1; geometry collision cylinder length=0.005 radius=0.15; visual mesh filename=package://hola_bot/meshes/base_link.obj
- link front_wheel: mass 0.062 -> 0.060
Joints:
- removed joint back_left_joint
- removed joint back_right_joint
- added joint left_joint: type revolute, parent base_link, child left_wheel, origin xyz=-0.15154 -0.087275 0 rpy=0 0 2.094, axis 0 1 0, limit effort=5 velocity=5
- added joint right_joint: type revolute, parent base_link, child right_wheel, origin xyz=0.15154 -0.087275 0 rpy=0 0 -2.094, axis 0 1 0, limit effort=5 velocity=5
- joint front_joint: origin xyz=0 0.17483 -0.0335 rpy=0 0 0 -> xyz=0 0.17483 0 rpy=0 0 0; type continuous -> revolute
